File: case/avia Mk1/base/Base.kicad_pcb (KiCad board)
At the start: 2 copper layers, 43.5 x 51.1 mm, 1 part

Commit message: small corrections
Other:
- board text added: "avia Mk1"
- board text added: "avia base v1.0"
- board text removed: "libra Mk8 navigator Watch base"
- board text removed: "libra navigator Mk8"
Changed lines of the file:
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@@
       (drillshape 0)
       (scaleselection 1)
-      (outputdirectory "output/base/")
+      (outputdirectory "out/")
     )
   )
@@
     (effects (font (size 2.5 2.5) (thickness 0.3)) (justify mirror))
   )
-  (gr_text "libra navigator Mk8" (at 144.06 76.81) (layer "B.SilkS")
+  (gr_text "avia Mk1" (at 144.06 76.81) (layer "B.SilkS")
     (effects (font (size 1 1.4) (thickness 0.2)) (justify mirror))
   )
@@
     (effects (font (size 1.5 1.5) (thickness 0.15)) (justify mirror))
   )
-  (gr_text "libra Mk8 navigator\nWatch base" (at 137.8 89.18) (layer "F.SilkS")
+  (gr_text "avia base v1.0" (at 137.8 89.18) (layer "F.SilkS")
     (effects (font (size 0.6 1) (thickness 0.15)) (justify left))
   )
