File: case/avia Mk1/slider/slider.kicad_pcb (KiCad board)
At the start: 2 copper layers, 30.9 x 30.9 mm, 0 parts

Commit message: small corrections
Other:
- outline, holes or cut-outs redrawn
- board text added: "avia slider v1.0"
Changed lines of the file:
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@@
     (pad_to_mask_clearance 0)
     (pcbplotparams
-      (layerselection 0x00010fc_ffffffff)
+      (layerselection 0x0000020_7ffffffe)
       (disableapertmacros false)
       (usegerberextensions false)
@@
       (svguseinch false)
       (svgprecision 6)
-      (excludeedgelayer true)
+      (excludeedgelayer false)
       (plotframeref false)
       (viasonmask false)
@@
       (dxfimperialunits true)
       (dxfusepcbnewfont true)
-      (psnegative false)
+      (psnegative true)
       (psa4output false)
       (plotreference true)
@@
       (sketchpadsonfab false)
       (subtractmaskfromsilk false)
-      (outputformat 1)
+      (outputformat 4)
       (mirror false)
       (drillshape 0)
       (scaleselection 1)
-      (outputdirectory "output/ring/")
+      (outputdirectory "out/")
     )
   )
@@
   (gr_line (start 151.14 79.65) (end 150.77 80.51) (layer "F.SilkS") (width 0.12))
   (gr_line (start 151.51 80.51) (end 151.14 79.65) (layer "F.SilkS") (width 0.12))
-  (gr_circle (center 151.14 95.1) (end 164.64 95.1) (layer "Edge.Cuts") (width 0.1) (fill none))
+  (gr_line (start 156.35 108.57) (end 155.77 108.77) (layer "Edge.Cuts") (width 0.05))
+  (gr_line (start 155.77 108.77) (end 155.46 107.89) (layer "Edge.Cuts") (width 0.05))
+  (gr_line (start 143.23 107.16) (end 142.74 106.87) (layer "Edge.Cuts") (width 0.05))
+  (gr_arc (start 143.3 106.089999) (mid 137.745961 93.413172) (end 146.269724 82.509286) (layer "Edge.Cuts") (width 0.05))
+  (gr_arc (start 158.98 84.110001) (mid 164.534039 96.786828) (end 156.010276 107.690714) (layer "Edge.Cuts") (width 0.05))
+  (gr_arc (start 146.82 82.31) (mid 152.851656 81.70908) (end 158.538232 83.80785) (layer "Edge.Cuts") (width 0.05))
+  (gr_line (start 146.51 81.43) (end 146.82 82.31) (layer "Edge.Cuts") (width 0.05))
+  (gr_line (start 159.05 83.04) (end 159.54 83.33) (layer "Edge.Cuts") (width 0.05))
+  (gr_line (start 143.23 107.16) (end 143.741677 106.392289) (layer "Edge.Cuts") (width 0.05))
+  (gr_line (start 146.27 82.51) (end 145.93 81.63) (layer "Edge.Cuts") (width 0.05))
+  (gr_line (start 156.01 107.69) (end 156.35 108.57) (layer "Edge.Cuts") (width 0.05))
+  (gr_line (start 145.93 81.63) (end 146.51 81.43) (layer "Edge.Cuts") (width 0.05))
+  (gr_line (start 142.74 106.87) (end 143.3 106.09) (layer "Edge.Cuts") (width 0.05))
   (gr_circle (center 151.14 95.1) (end 166.6 95.1) (layer "Edge.Cuts") (width 0.1) (fill none))
+  (gr_line (start 159.54 83.33) (end 158.98 84.11) (layer "Edge.Cuts") (width 0.05))
+  (gr_arc (start 155.46 107.89) (mid 149.428344 108.49092) (end 143.741768 106.39215) (layer "Edge.Cuts") (width 0.05))
+  (gr_line (start 159.05 83.04) (end 158.538323 83.807711) (layer "Edge.Cuts") (width 0.05))
   (gr_circle (center 151.14 95.1) (end 151.2 95.1) (layer "User.2") (width 0.1) (fill none))
   (gr_line (start 165.373038 88.763043) (end 164.834046 89.003018) (layer "User.3") (width 0.1))
@@
   (gr_line (start 166.552863 92.824026) (end 165.969192 92.910215) (layer "User.3") (width 0.1))
   (gr_line (start 138.535515 104.257694) (end 139.012835 103.910901) (layer "User.3") (width 0.1))
+  (gr_text "avia slider v1.0" (at 151.37 80.6) (layer "B.SilkS")
+    (effects (font (size 0.6 0.6) (thickness 0.12)) (justify mirror))
+  )
   (gr_text "|" (at 159.73 82.72 -34.82) (layer "F.SilkS")
     (effects (font (size 0.6 1) (thickness 0.125)))
