File: case/avia Mk2/current/inner dial/inner.kicad_pcb (KiCad board)
At the start: 2 copper layers, 39.8 x 39.8 mm, 1 part

Commit message: v0.2 case
Parts:
- removed G***: LOGO, BartLib_Logo:BD_small 3.5x2.6
Routing:
- net (no net): vias 4 -> 0
Other:
- board text removed: "Mk1"
