File: case/avia Mk2/snapshots/16 fixed bottom telescope/current/outer dial/outer.kicad_pcb (KiCad board)
At the start: 2 copper layers, 48 x 48 mm, 0 parts

Commit message: v0.2 case
Other:
- board text added: "avia slider v1.0"
- board text removed: "avia slider v2.0"
