File: case/avia Mk2/current/cover/cover.kicad_pcb (KiCad board)
At the start: 2 copper layers, 48.4 x 46.8 mm, 1 part

Commit message: version with case renamed to Mk2
Other:
- board text added: "avia Mk2"
- board text removed: "avia Mk1"
Changed lines of the file:
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@@
   (gr_line (start 166.19 100) (end 232.37 100) (layer "User.1") (width 0.1))
   (gr_circle (center 200 100) (end 199.298858 100) (layer "User.1") (width 1) (fill none))
-  (gr_text "avia Mk1" (at 200.113504 82.57) (layer "F.SilkS")
+  (gr_text "avia Mk2" (at 200.113504 82.57) (layer "F.SilkS")
     (effects (font (size 1 1.4) (thickness 0.2)))
   )
