File: pcb/sense_slim/sense_slim.kicad_pcb (KiCad board)
At the start: 2 copper layers, 44 x 42.5 mm, 75 parts, among them J1 PFC24/display, J2 USB_B_Micro, J3 programming, J5 START, J6 SET, J7 RESET, Q1 IRLML0030TR, Q2 PMBTA14,215, Q3 PMBTA14,215, Q4 PMBTA14,215, U1 BME280, U2 STM32G071KxT, U3 TC1185-3.3, U4 MCP73831-2-OT, U5 LIS3MDL, Y1 32k768

Commit message: added forecast icons
Parts:
- C1, C17, C18: value 225 -> 2u2
- C10, C11, C12, C13, C14, C15, C16, C27: value 105 -> 1u
- C19, C20, C29: value 475 -> 4u7
- C2, C21, C25, C26, C30, C9: value 104 -> 100n
- C22, C23, C24: value 222 -> 2n2
- C3, C4: value 100 -> 10p
- C5, C6: value 475 50V -> 4u7 50V
- Q2, Q3, Q4: value PMBTA14,215 -> BCV27.215
- R10, R12, R13, R14, R18, R8: value 100k -> 1k
- R19, R20, R21: value 39k -> 1k
- R9: value 470R -> 10k
Connections:
- U2 pad 12: /OHMOMETER -> unconnected-(U2-Pad12)
- U2 pad 7: /VOLTIMETER -> unconnected-(U2-Pad7)
