File: pcb/sense_slim/sense_slim.kicad_sch (KiCad schematic)
At the start: 74 parts, among them J1 PFC24/display, J2 USB_B_Micro, J3 programming, J5 START, J6 SET, J7 RESET, Q1 IRLML0030TR, Q2 BCV27.215, Q3 BCV27.215, Q4 BCV27.215, U1 BME280, U2 STM32G071KxT, U3 TC1185-3.3, U4 MCP73831-2-OT, U5 LIS3MDL, Y1 32k768

Commit message: added forecast icons
Parts:
- C1, C17, C18: value 225 -> 2u2
- C10, C11, C12, C13, C14, C15, C16, C27: value 105 -> 1u
- C19, C20, C29: value 475 -> 4u7
- C2, C21, C25, C26, C30, C9: value 104 -> 100n
- C22, C23, C24: value 222 -> 2n2
- C3, C4: value 100 -> 10p
- C5, C6: value 475 50V -> 4u7 50V
- R10, R12, R13, R14, R18, R8: value 100k -> 1k
- R19, R20, R21: value 39k -> 1k
Connections:
- net OHMOMETER: no longer names the net of U2.12 (PA5)
- net VOLTIMETER: no longer names the net of U2.7 (PA0)
- no-connect marks 18 -> 21
Other:
- moved on the sheet: BT1, C17, C18, C19, C20, C29, C3, C30, C4, D4, D5, J2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

Commit message: fixed symbols
Parts:
- removed J2: USB_B_Micro, Connector_USB:USB_Micro-B_Molex_47346-0001, symbol sense-rescue:USB_B_Micro-Connector-venom-rescue
- removed U5: LIS3MDL, Package_LGA:LGA-12_2x2mm_P0.5mm, symbol sense-rescue:LIS3MDL-Venom
- added J2: USB_B_Micro, Connector_USB:USB_Micro-B_Molex_47346-0001, symbol Connector:USB_B_Micro
- added U5: LIS3MDL, Package_LGA:LGA-12_2x2mm_P0.5mm, symbol BartLib_Sensors:LIS3MDL
Connections:
- net +3V3: now also U5.10 (CS), U5.5 (Vdd), U5.6 (Vdd_IO)
- net GND: now also J2.5 (GND), J2.6 (Shield), U5.12 (RES), U5.2 (RES), U5.3 (GND), U5.9 (SDO/SA1)
- net SCL: now also U5.1 (SCL/SPC)
- net SDA: now also U5.11 (SDA/SDI/SDO)
- net at C19.1, D5.2 (A), U4.4 (VDD): now also J2.1 (VBUS)
- net at C25.1: now also U5.4 (C1)
Other:
- moved on the sheet: C26, C27

Commit message: schemaric without ERC errors
Other:
- note added: "BS"
- note added: "BUSY"
- note added: "CS"
- note added: "DC"
- note added: "GDR"
- note added: "HLT_CTL"
- note added: "PREVGH"
- note added: "PREVGL"
- note added: "RESE"
- note added: "RST"
- note added: "SCLK"
- note added: "SDI"
- note added: "TSCL"
- note added: "TSDA"
- note added: "VCI"
- note added: "VCOM"
- note added: "VDD"
- note added: "VDDIO"
- note added: "VGH"
- note added: "VGL"
- note added: "VPP"
- note added: "VSH"
- note added: "VSL"
- note added: "VSS"
Changed lines of the file:
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@@
     (stroke (width 0) (type default) (color 0 0 0 0))
+  )
+  (text "VGH" (at 271.145 29.21 0)
+    (effects (font (size 1.27 1.27)) (justify left bottom))
+  )
+  (text "PREVGH" (at 271.145 69.85 0)
+    (effects (font (size 1.27 1.27)) (justify left bottom))
+  )
+  (text "GDR" (at 271.145 21.59 0)
+    (effects (font (size 1.27 1.27)) (justify left bottom))
+  )
+  (text "TSCL" (at 271.145 31.75 0)
+    (effects (font (size 1.27 1.27)) (justify left bottom))
+  )
+  (text "VDDIO" (at 271.145 54.61 0)
+    (effects (font (size 1.27 1.27)) (justify left bottom))
+  )
+  (text "PREVGL" (at 271.145 74.93 0)
+    (effects (font (size 1.27 1.27)) (justify left bottom))
+  )
+  (text "VGL" (at 271.145 26.67 0)
+    (effects (font (size 1.27 1.27)) (justify left bottom))
+  )
+  (text "BUSY" (at 271.145 39.37 0)
+    (effects (font (size 1.27 1.27)) (justify left bottom))
+  )
+  (text "CS" (at 271.145 46.99 0)
+    (effects (font (size 1.27 1.27)) (justify left bottom))
+  )
+  (text "VSL" (at 271.145 72.39 0)
+    (effects (font (size 1.27 1.27)) (justify left bottom))
+  )
+  (text "VSS" (at 271.145 59.69 0)
+    (effects (font (size 1.27 1.27)) (justify left bottom))
   )
   (text "Connector: MOLEX PicoBlade\n*socket: 532610571\n*plug: 510210500\n*pin: 500798000"
@@
     (effects (font (size 1.27 1.27)) (justify left bottom))
   )
+  (text "SCLK" (at 271.145 49.53 0)
+    (effects (font (size 1.27 1.27)) (justify left bottom))
+  )
+  (text "VSH" (at 271.145 67.31 0)
+    (effects (font (size 1.27 1.27)) (justify left bottom))
+  )
+  (text "BS" (at 271.145 36.83 0)
+    (effects (font (size 1.27 1.27)) (justify left bottom))
+  )
+  (text "VCOM" (at 271.145 77.47 0)
+    (effects (font (size 1.27 1.27)) (justify left bottom))
+  )
   (text "CATHODE PROTECTION" (at 19.685 88.265 0)
     (effects (font (size 1.27 1.27)) (justify left bottom))
   )
+  (text "VDD" (at 271.145 62.23 0)
+    (effects (font (size 1.27 1.27)) (justify left bottom))
+  )
   (text "ALL DISPLAY CAPACITORS 50V" (at 219.075 107.95 0)
     (effects (font (size 1.27 1.27)) (justify left bottom))
   )
+  (text "TSDA" (at 271.145 34.29 0)
+    (effects (font (size 1.27 1.27)) (justify left bottom))
+  )
+  (text "RST" (at 271.145 41.91 0)
+    (effects (font (size 1.27 1.27)) (justify left bottom))
+  )
+  (text "VPP" (at 271.145 64.77 0)
+    (effects (font (size 1.27 1.27)) (justify left bottom))
+  )
+  (text "HLT_CTL" (at 271.145 19.05 0)
+    (effects (font (size 1.27 1.27)) (justify left bottom))
+  )
+  (text "VCI" (at 271.145 57.15 0)
+    (effects (font (size 1.27 1.27)) (justify left bottom))
+  )
+  (text "DC" (at 271.145 44.45 0)
+    (effects (font (size 1.27 1.27)) (justify left bottom))
+  )
+  (text "RESE" (at 271.145 24.13 0)
+    (effects (font (size 1.27 1.27)) (justify left bottom))
+  )
+  (text "SDI" (at 271.145 52.07 0)
+    (effects (font (size 1.27 1.27)) (justify left bottom))
+  )
   (label "BUSY" (at 241.935 39.37 0)
     (effects (font (size 1.27 1.27)) (justify left bottom))
@@
     (effects (font (size 1.27 1.27)) (justify left bottom))
   )
-  (label "PREVGL" (at 271.145 74.93 0)
-    (effects (font (size 1.27 1.27)) (justify left bottom))
-  )
   (label "SDA" (at 55.88 158.115 0)
     (effects (font (size 1.27 1.27)) (justify left bottom))
@@
     (effects (font (size 1.27 1.27)) (justify right bottom))
   )
-  (label "TSDA" (at 271.145 34.29 0)
-    (effects (font (size 1.27 1.27)) (justify left bottom))
-  )
   (label "SWDIO" (at 20.32 173.355 180)
     (effects (font (size 1.27 1.27)) (justify right bottom))
   )
-  (label "VSS" (at 271.145 59.69 0)
-    (effects (font (size 1.27 1.27)) (justify left bottom))
-  )
   (label "SWDRST" (at 57.785 178.435 0)
     (effects (font (size 1.27 1.27)) (justify left bottom))
   )
-  (label "VGL" (at 271.145 26.67 0)
-    (effects (font (size 1.27 1.27)) (justify left bottom))
-  )
   (label "SDA" (at 92.075 33.02 180)
     (effects (font (size 1.27 1.27)) (justify right bottom))
@@
     (effects (font (size 1.27 1.27)) (justify left bottom))
   )
-  (label "TSCL" (at 271.145 31.75 0)
-    (effects (font (size 1.27 1.27)) (justify left bottom))
-  )
   (label "START" (at 20.32 145.415 180)
     (effects (font (size 1.27 1.27)) (justify right bottom))
@@
     (effects (font (size 1.27 1.27)) (justify right bottom))
   )
-  (label "PREVGH" (at 271.145 69.85 0)
-    (effects (font (size 1.27 1.27)) (justify left bottom))
-  )
   (label "MOSI" (at 241.935 52.07 0)
     (effects (font (size 1.27 1.27)) (justify left bottom))
@@
     (effects (font (size 1.27 1.27)) (justify right bottom))
   )
-  (label "RST" (at 271.145 41.91 0)
-    (effects (font (size 1.27 1.27)) (justify left bottom))
-  )
   (label "RST" (at 20.32 165.735 180)
     (effects (font (size 1.27 1.27)) (justify right bottom))
@@
     (effects (font (size 1.27 1.27)) (justify right bottom))
   )
-  (label "VSL" (at 271.145 72.39 0)
-    (effects (font (size 1.27 1.27)) (justify left bottom))
-  )
   (label "SCL" (at 88.265 33.02 180)
     (effects (font (size 1.27 1.27)) (justify right bottom))
@@
     (effects (font (size 1.27 1.27)) (justify left bottom))
   )
-  (label "VGH" (at 271.145 29.21 0)
-    (effects (font (size 1.27 1.27)) (justify left bottom))
-  )
   (label "SWDCLK" (at 66.675 92.075 0)
     (effects (font (size 1.27 1.27)) (justify left bottom))
@@
     (effects (font (size 1.27 1.27)) (justify right bottom))
   )
-  (label "VDDIO" (at 271.145 54.61 0)
-    (effects (font (size 1.27 1.27)) (justify left bottom))
-  )
-  (label "SDI" (at 271.145 52.07 0)
-    (effects (font (size 1.27 1.27)) (justify left bottom))
-  )
-  (label "RESE" (at 271.145 24.13 0)
-    (effects (font (size 1.27 1.27)) (justify left bottom))
-  )
   (label "VIN" (at 19.685 76.835 0)
     (effects (font (size 1.27 1.27)) (justify left bottom))
@@
     (effects (font (size 1.27 1.27)) (justify left bottom))
   )
-  (label "VDD" (at 271.145 62.23 0)
-    (effects (font (size 1.27 1.27)) (justify left bottom))
-  )
   (label "RESE" (at 257.175 24.13 0)
     (effects (font (size 1.27 1.27)) (justify left bottom))
@@
     (effects (font (size 1.27 1.27)) (justify left bottom))
   )
-  (label "BUSY" (at 271.145 39.37 0)
-    (effects (font (size 1.27 1.27)) (justify left bottom))
-  )
   (label "RESET" (at 20.32 150.495 180)
     (effects (font (size 1.27 1.27)) (justify right bottom))
@@
     (effects (font (size 1.27 1.27)) (justify left bottom))
   )
-  (label "GDR" (at 271.145 21.59 0)
-    (effects (font (size 1.27 1.27)) (justify left bottom))
-  )
   (label "PREVGL" (at 194.945 24.13 0)
     (effects (font (size 1.27 1.27)) (justify left bottom))
@@
     (effects (font (size 1.27 1.27)) (justify right bottom))
   )
-  (label "VPP" (at 271.145 64.77 0)
-    (effects (font (size 1.27 1.27)) (justify left bottom))
-  )
-  (label "SCLK" (at 271.145 49.53 0)
-    (effects (font (size 1.27 1.27)) (justify left bottom))
-  )
-  (label "CS" (at 271.145 46.99 0)
-    (effects (font (size 1.27 1.27)) (justify left bottom))
-  )
   (label "START" (at 149.225 97.79 180)
     (effects (font (size 1.27 1.27)) (justify right bottom))
   )
-  (label "VCI" (at 271.145 57.15 0)
-    (effects (font (size 1.27 1.27)) (justify left bottom))
-  )
-  (label "DC" (at 271.145 44.45 0)
-    (effects (font (size 1.27 1.27)) (justify left bottom))
-  )
   (label "CS" (at 241.935 46.99 0)
     (effects (font (size 1.27 1.27)) (justify left bottom))
@@
     (effects (font (size 1.27 1.27)) (justify right bottom))
   )
-  (label "BS" (at 271.145 36.83 0)
-    (effects (font (size 1.27 1.27)) (justify left bottom))
-  )
-  (label "VCOM" (at 271.145 77.47 0)
-    (effects (font (size 1.27 1.27)) (justify left bottom))
-  )
   (label "PREVGH" (at 244.475 69.85 180)
     (effects (font (size 1.27 1.27)) (justify right bottom))
@@
     (effects (font (size 1.27 1.27)) (justify right bottom))
   )
-  (label "HLT_CTL" (at 271.145 19.05 0)
-    (effects (font (size 1.27 1.27)) (justify left bottom))
-  )
-  (label "VSH" (at 271.145 67.31 0)
-    (effects (font (size 1.27 1.27)) (justify left bottom))
-  )
   (label "SET" (at 149.225 135.89 180)
